File: chronos-polaris-hardware/Dual-PNP-Small-Signal-Transistor_sch.kicad_sch (KiCad schematic)
At the start: 7 parts, among them U13 2N7002KDW_72K, U4 AP20P30Q, U6 AP20P30Q

Commit message: clean up
Parts:
- renumbered R23 to R?, R21 to R?, R22 to R?, R27 to R?, U6 to U?, U4 to U?, U13 to U?
Changed lines of the file:
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@@
 		(dnp no)
 		(fields_autoplaced yes)
-		(property "Reference" "#PWR050"
+		(property "Reference" "#PWR?"
 			(at 144.78 95.25 0)
 			(effects
@@
 		(pin "1"
 		)
+		(instances
+			(project "chronos-polaris-hardware"
+				(path "/503f01d5-a0c6-4ade-b485-97c3c2e1d6c5/8b4919a7-1d2e-4328-8834-b08438b11cfd"
+					(reference "#PWR?")
+					(unit 1)
+				)
+			)
+		)
 	)
 	(symbol
@@
 		(dnp no)
 		(fields_autoplaced yes)
-		(property "Reference" "U6"
+		(property "Reference" "U?"
 			(at 128.27 70.485 0)
 			(effects
@@
 		(pin "9"
 		)
+		(instances
+			(project "chronos-polaris-hardware"
+				(path "/503f01d5-a0c6-4ade-b485-97c3c2e1d6c5/8b4919a7-1d2e-4328-8834-b08438b11cfd"
+					(reference "U?")
+					(unit 1)
+				)
+			)
+		)
 	)
 	(symbol
@@
 		(on_board yes)
 		(dnp no)
-		(property "Reference" "R23"
+		(property "Reference" "R?"
 			(at 167.64 62.23 0)
 			(effects
@@
 		(pin "2"
 		)
+		(instances
+			(project "chronos-polaris-hardware"
+				(path "/503f01d5-a0c6-4ade-b485-97c3c2e1d6c5/8b4919a7-1d2e-4328-8834-b08438b11cfd"
+					(reference "R?")
+					(unit 1)
+				)
+			)
+		)
 	)
 	(symbol
@@
 		(dnp no)
 		(fields_autoplaced yes)
-		(property "Reference" "#PWR053"
+		(property "Reference" "#PWR?"
 			(at 154.94 109.22 0)
 			(effects
@@
 		(pin "1"
 		)
+		(instances
+			(project "chronos-polaris-hardware"
+				(path "/503f01d5-a0c6-4ade-b485-97c3c2e1d6c5/8b4919a7-1d2e-4328-8834-b08438b11cfd"
+					(reference "#PWR?")
+					(unit 1)
+				)
+			)
+		)
 	)
 	(symbol
@@
 		(on_board yes)
 		(dnp no)
-		(property "Reference" "R21"
+		(property "Reference" "R?"
 			(at 138.43 83.82 0)
 			(effects
@@
 		(pin "2"
 		)
+		(instances
+			(project "chronos-polaris-hardware"
+				(path "/503f01d5-a0c6-4ade-b485-97c3c2e1d6c5/8b4919a7-1d2e-4328-8834-b08438b11cfd"
+					(reference "R?")
+					(unit 1)
+				)
+			)
+		)
 	)
 	(symbol
@@
 		(on_board yes)
 		(dnp no)
-		(property "Reference" "#PWR052"
+		(property "Reference" "#PWR?"
 			(at 163.83 53.34 0)
 			(effects
@@
 		(pin "1"
 		)
+		(instances
+			(project "chronos-polaris-hardware"
+				(path "/503f01d5-a0c6-4ade-b485-97c3c2e1d6c5/8b4919a7-1d2e-4328-8834-b08438b11cfd"
+					(reference "#PWR?")
+					(unit 1)
+				)
+			)
+		)
 	)
 	(symbol
@@
 		(dnp no)
 		(fields_autoplaced yes)
-		(property "Reference" "#PWR051"
+		(property "Reference" "#PWR?"
 			(at 149.86 67.31 0)
 			(effects
@@
 		(pin "1"
 		)
+		(instances
+			(project "chronos-polaris-hardware"
+				(path "/503f01d5-a0c6-4ade-b485-97c3c2e1d6c5/8b4919a7-1d2e-4328-8834-b08438b11cfd"
+					(reference "#PWR?")
+					(unit 1)
+				)
+			)
+		)
 	)
 	(symbol
@@
 		(dnp no)
 		(fields_autoplaced yes)
-		(property "Reference" "U4"
+		(property "Reference" "U?"
 			(at 124.46 89.535 0)
 			(effects
@@
 		(pin "9"
 		)
+		(instances
+			(project "chronos-polaris-hardware"
+				(path "/503f01d5-a0c6-4ade-b485-97c3c2e1d6c5/8b4919a7-1d2e-4328-8834-b08438b11cfd"
+					(reference "U?")
+					(unit 1)
+				)
+			)
+		)
 	)
 	(symbol
@@
 		(dnp no)
 		(fields_autoplaced yes)
-		(property "Reference" "R22"
+		(property "Reference" "R?"
 			(at 147.32 64.135 0)
 			(effects
@@
 		(pin "2"
 		)
+		(instances
+			(project "chronos-polaris-hardware"
+				(path "/503f01d5-a0c6-4ade-b485-97c3c2e1d6c5/8b4919a7-1d2e-4328-8834-b08438b11cfd"
+					(reference "R?")
+					(unit 1)
+				)
+			)
+		)
 	)
 	(symbol
@@
 		(dnp no)
 		(fields_autoplaced yes)
-		(property "Reference" "U13"
+		(property "Reference" "U?"
 			(at 153.67 80.645 90)
 			(effects
@@
 		(pin "6"
 		)
+		(instances
+			(project "chronos-polaris-hardware"
+				(path "/503f01d5-a0c6-4ade-b485-97c3c2e1d6c5/8b4919a7-1d2e-4328-8834-b08438b11cfd"
+					(reference "U?")
+					(unit 1)
+				)
+			)
+		)
 	)
 	(symbol
@@
 		(dnp no)
 		(fields_autoplaced yes)
-		(property "Reference" "R27"
+		(property "Reference" "R?"
 			(at 157.48 98.425 0)
 			(effects
@@
 		(pin "2"
 		)
-	)
+		(instances
+			(project "chronos-polaris-hardware"
+				(path "/503f01d5-a0c6-4ade-b485-97c3c2e1d6c5/8b4919a7-1d2e-4328-8834-b08438b11cfd"
+					(reference "R?")
+					(unit 1)
+				)
+			)
+		)
+	)
