File: chronos-polaris-hardware/chronos-polaris-hardware.kicad_sch (KiCad schematic)
At the start: 30 parts, among them J1 Conn_01x03_Pin, J2 Conn_01x03_Pin, J3 Conn_01x03_Pin, J4 Conn_01x03_Pin, J5 Conn_01x03_Pin, J6 Conn_01x04, J7 Conn_01x04, J8 Conn_01x02, J9 691417320006S, Q1 US6K4TR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

Commit message: end it all
Parts:
- Q1: footprint US6K4TR -> KiCad:US6K4TR
Changed lines of the file:
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@@
 			)
 		)
-		(property "Footprint" "US6K4TR"
+		(property "Footprint" "KiCad:US6K4TR"
 			(at 104.14 205.41 0)
 			(effects

Commit message: finnaly
Parts:
- J9: footprint TerminalBlock_NEW_Wurth:691417320006S -> polaris-fp:691417320006S
Changed lines of the file:
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@@
 			)
 		)
-		(property "Footprint" "TerminalBlock_NEW_Wurth:691417320006S"
+		(property "Footprint" "polaris-fp:691417320006S"
 			(at 30.48 64.77 0)
 			(effects
@@
 	)
 	(symbol
+		(lib_id "polaris-sym:TF_PUSH")
+		(at 149.86 156.21 180)
+		(unit 1)
+		(exclude_from_sim no)
+		(in_bom yes)
+		(on_board yes)
+		(dnp no)
+		(fields_autoplaced yes)
+		(property "Reference" "U5"
+			(at 135.89 154.9399 0)
+			(effects
+				(font
+					(size 1.27 1.27)
+				)
+				(justify left)
+			)
+		)
+		(property "Value" "TF_PUSH"
+			(at 135.89 157.4799 0)
+			(effects
+				(font
+					(size 1.27 1.27)
+				)
+				(justify left)
+			)
+		)
+		(property "Footprint" "polaris-fp:TF-SMD_TF-PUSH"
+			(at 149.86 146.05 0)
+			(effects
+				(font
+					(size 1.27 1.27)
+					(italic yes)
+				)
+				(hide yes)
+			)
+		)
+		(property "Datasheet" "https://item.szlcsc.com/372553.html"
+			(at 152.146 156.337 0)
+			(effects
+				(font
+					(size 1.27 1.27)
+				)
+				(justify left)
+				(hide yes)
+			)
+		)
+		(property "Description" ""
+			(at 149.86 156.21 0)
+			(effects
+				(font
+					(size 1.27 1.27)
+				)
+				(hide yes)
+			)
+		)
+		(property "LCSC" "C393941"
+			(at 149.86 156.21 0)
+			(effects
+				(font
+					(size 1.27 1.27)
+				)
+				(hide yes)
+			)
+		)
+		(pin "3"
+		)
+		(pin "5"
+		)
+		(pin "10"
+		)
+		(pin "2"
+		)
+		(pin "6"
+		)
+		(pin "11"
+		)
+		(pin "7"
+		)
+		(pin "13"
+		)
+		(pin "1"
+		)
+		(pin "4"
+		)
+		(pin "8"
+		)
+		(pin "9"
+		)
+		(pin "12"
+		)
+		(instances
+			(project ""
+				(path "/503f01d5-a0c6-4ade-b485-97c3c2e1d6c5"
+					(reference "U5")
+					(unit 1)
+				)
+			)
+		)
+	)
+	(symbol
 		(lib_name "GND_1")
 		(lib_id "power:GND")
@@
 					(unit 1)
 				)
-			)
-		)
-	)
-	(symbol
-		(lib_id "polaris-sym:TF_PUSH")
-		(at 149.86 156.21 180)
-		(unit 1)
-		(exclude_from_sim no)
-		(in_bom yes)
-		(on_board yes)
-		(dnp no)
-		(fields_autoplaced yes)
-		(property "Reference" "U5"
-			(at 135.89 156.845 0)
-			(effects
-				(font
-					(size 1.27 1.27)
-				)
-				(justify left)
-			)
-		)
-		(property "Value" "TF_PUSH"
-			(at 135.89 154.305 0)
-			(effects
-				(font
-					(size 1.27 1.27)
-				)
-				(justify left)
-			)
-		)
-		(property "Footprint" "polaris-fp:TF-SMD_TF-PUSH"
-			(at 149.86 146.05 0)
-			(effects
-				(font
-					(size 1.27 1.27)
-					(italic yes)
-				)
-				(hide yes)
-			)
-		)
-		(property "Datasheet" "https://item.szlcsc.com/372553.html"
-			(at 152.146 156.337 0)
-			(effects
-				(font
-					(size 1.27 1.27)
-				)
-				(justify left)
-				(hide yes)
-			)
-		)
-		(property "Description" ""
-			(at 149.86 156.21 0)
-			(effects
-				(font
-					(size 1.27 1.27)
-				)
-				(hide yes)
-			)
-		)
-		(property "LCSC" "C393941"
-			(at 149.86 156.21 0)
-			(effects
-				(font
-					(size 1.27 1.27)
-				)
-				(hide yes)
-			)
-		)
-		(pin "1"
-		)
-		(pin "10"
-		)
-		(pin "11"
-		)
-		(pin "12"
-		)
-		(pin "13"
-		)
-		(pin "2"
-		)
-		(pin "3"
-		)
-		(pin "4"
-		)
-		(pin "5"
-		)
-		(pin "6"
-		)
-		(pin "7"
-		)
-		(pin "8"
-		)
-		(pin "9"
-		)
-		(instances
-			(project "chronos-polaris-hardware"
-				(path "/503f01d5-a0c6-4ade-b485-97c3c2e1d6c5"
-					(reference "U5")
-					(unit 1)
-				)

Commit message: abcd
Parts:
- added J10: TSW-102-07-G-D, rigelcon:TSW-102-07-G-D_SAI, symbol rigelcon:TSW-102-07-G-D
Changed lines of the file:
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@@
+	)
+	(symbol
+		(lib_id "rigelcon:TSW-102-07-G-D")
+		(at 49.53 31.75 0)
+		(unit 1)
+		(exclude_from_sim no)
+		(in_bom yes)
+		(on_board yes)
+		(dnp no)
+		(fields_autoplaced yes)
+		(property "Reference" "J10"
+			(at 69.85 21.59 0)
+			(effects
+				(font
+					(size 1.524 1.524)
+				)
+			)
+		)
+		(property "Value" "TSW-102-07-G-D"
+			(at 69.85 24.13 0)
+			(effects
+				(font
+					(size 1.524 1.524)
+				)
+			)
+		)
+		(property "Footprint" "rigelcon:TSW-102-07-G-D_SAI"
+			(at 49.53 31.75 0)
+			(effects
+				(font
+					(size 1.27 1.27)
+					(italic yes)
+				)
+				(hide yes)
+			)
+		)
+		(property "Datasheet" "TSW-102-07-G-D"
+			(at 49.53 31.75 0)
+			(effects
+				(font
+					(size 1.27 1.27)
+					(italic yes)
+				)
+				(hide yes)
+			)
+		)
+		(property "Description" ""
+			(at 49.53 31.75 0)
+			(effects
+				(font
+					(size 1.27 1.27)
+				)
+				(hide yes)
+			)
+		)
+		(pin "4"
+		)
+		(pin "3"
+		)
+		(pin "1"
+		)
+		(pin "2"
+		)
+		(instances
+			(project ""
+				(path "/503f01d5-a0c6-4ade-b485-97c3c2e1d6c5"
+					(reference "J10")
+					(unit 1)
+				)
+			)
+		)
 	)
 	(symbol
