File: chronos-polaris-hardware/chronos-polaris-hardware-revised.kicad_pcb (KiCad board)
At the start: 2 copper layers, 66 parts, among them J1 Conn_01x03_Pin, J10 TSW-102-07-G-D, J2 Conn_01x03_Pin, J3 Conn_01x03_Pin, J4 Conn_01x03_Pin, J5 Conn_01x03_Pin, J6 Conn_01x04, J7 Conn_01x04, J8 Conn_01x02, J9 691417320006S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

Commit message: Added Direct Datasheet Links
(except for pressure sensor AMP2167, I couldn't find a pdf datasheet)
Parts:
- U2: value ESP32 -> ESP32-S2-SOLO-2-N4
Connections:
- J10 pad 1: /DROGUE DETECT -> Rigel1
- U2 pad 16: /DROGUE DETECT -> Rigel1
